File: examples/SkyKey-AT42QT1011.kicad_sch (KiCad schematic)
At the start: 7 parts, among them J2 SkyKey, U2 AT42QT1011-TSHR

Commit message: Fix examples
Parts:
- renumbered C7 to C10, C8 to C11, D102 to D103, J2 to J3, KS4 to KS6, R4 to R6, U2 to U3
