File: examples/SkySense-bank.kicad_sch (KiCad schematic)
At the start: 4 parts

Commit message: Fix examples
Parts:
- renumbered C1 to C501, C2 to C502, FB1 to FB501, FB2 to FB502
Changed lines of the file:
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@@
 		(in_pos_files yes)
 		(dnp no)
-		(property "Reference" "#PWR03"
+		(property "Reference" "#PWR0501"
 			(at 45.72 43.18 0)
 			(hide yes)
@@
 				(path "/a2fa3ed2-fc05-4238-b3b8-c73f0b2cdc77"
 					(reference "#PWR0501")
-					(unit 1)
-				)
-				(path "/a2fa3ed2-fc05-4238-b3b8-c73f0b2cdc77/00000000-0000-0000-0000-000060931a6c"
-					(reference "#PWR?")
-					(unit 1)
-				)
-				(path "/a2fa3ed2-fc05-4238-b3b8-c73f0b2cdc77/00000000-0000-0000-0000-00006095a3e7"
-					(reference "#PWR?")
-					(unit 1)
-				)
-				(path "/a2fa3ed2-fc05-4238-b3b8-c73f0b2cdc77/00000000-0000-0000-0000-00006095a595"
-					(reference "#PWR?")
-					(unit 1)
-				)
-				(path "/a2fa3ed2-fc05-4238-b3b8-c73f0b2cdc77/00000000-0000-0000-0000-00006095a623"
-					(reference "#PWR?")
-					(unit 1)
-				)
-				(path "/a2fa3ed2-fc05-4238-b3b8-c73f0b2cdc77/00000000-0000-0000-0000-00006097747f"
-					(reference "#PWR?")
-					(unit 1)
-				)
-				(path "/a2fa3ed2-fc05-4238-b3b8-c73f0b2cdc77/00000000-0000-0000-0000-00006097748e"
-					(reference "#PWR?")
 					(unit 1)
 				)
@@
 		(in_pos_files yes)
 		(dnp no)
-		(property "Reference" "C1"
+		(property "Reference" "C501"
 			(at 59.4868 43.2816 0)
 			(show_name no)
@@
 		(in_pos_files yes)
 		(dnp no)
-		(property "Reference" "#PWR05"
+		(property "Reference" "#PWR0502"
 			(at 45.72 55.88 0)
 			(hide yes)
@@
 				(path "/a2fa3ed2-fc05-4238-b3b8-c73f0b2cdc77"
 					(reference "#PWR0502")
-					(unit 1)
-				)
-				(path "/a2fa3ed2-fc05-4238-b3b8-c73f0b2cdc77/00000000-0000-0000-0000-000060931a6c"
-					(reference "#PWR?")
-					(unit 1)
-				)
-				(path "/a2fa3ed2-fc05-4238-b3b8-c73f0b2cdc77/00000000-0000-0000-0000-00006095a3e7"
-					(reference "#PWR?")
-					(unit 1)
-				)
-				(path "/a2fa3ed2-fc05-4238-b3b8-c73f0b2cdc77/00000000-0000-0000-0000-00006095a595"
-					(reference "#PWR?")
-					(unit 1)
-				)
-				(path "/a2fa3ed2-fc05-4238-b3b8-c73f0b2cdc77/00000000-0000-0000-0000-00006095a623"
-					(reference "#PWR?")
-					(unit 1)
-				)
-				(path "/a2fa3ed2-fc05-4238-b3b8-c73f0b2cdc77/00000000-0000-0000-0000-00006097747f"
-					(reference "#PWR?")
-					(unit 1)
-				)
-				(path "/a2fa3ed2-fc05-4238-b3b8-c73f0b2cdc77/00000000-0000-0000-0000-00006097748e"
-					(reference "#PWR?")
 					(unit 1)
 				)
@@
 		(in_pos_files yes)
 		(dnp no)
-		(property "Reference" "#PWR06"
+		(property "Reference" "#PWR0503"
 			(at 57.15 55.88 0)
 			(hide yes)
@@
 		(in_pos_files yes)
 		(dnp no)
-		(property "Reference" "FB2"
+		(property "Reference" "FB502"
 			(at 52.07 43.5102 90)
 			(show_name no)
@@
 		(in_pos_files yes)
 		(dnp no)
-		(property "Reference" "FB1"
+		(property "Reference" "FB501"
 			(at 50.8 34.6202 90)
 			(show_name no)
@@
 		(in_pos_files yes)
 		(dnp no)
-		(property "Reference" "C2"
+		(property "Reference" "C502"
 			(at 67.1068 43.2816 0)
 			(show_name no)
@@
 		)
 	)
+	(sheet_instances
+		(path "/"
+			(page "1")
+		)
+	)
+	(embedded_fonts no)
 )
